Commit message: asasas

File: intrarobots_ws/src/extras/extrernal_urdfs/camera_depth.xacro (robot description, xacro)
@@ -3,5 +3,6 @@
   <joint name="camera_joint" type="fixed">
       <axis xyz="0 1 0" />
-      <origin rpy="0 ${pi/2} 0" xyz="0 0.54 0.8" />
+      <!-- <origin rpy="0 ${pi/2} 0" xyz="0 0.54 0.8" /> -->
+      <origin rpy="${pi} ${3*pi/4} 0" xyz="0.4 0.3 0.35" />
       <!--parent link fixed-->
       <!-- <parent link="$(arg robot_name)/base_link"/> -->
