Commit message: asasas

File: intrarobots_ws/src/master/extrernal_urdfs/camera.xacro (robot description, xacro)
@@ -6,5 +6,5 @@
       <!--parent link fixed-->
       <!-- <parent link="$(arg robot_name)/base_link"/> -->
-      <parent link="panda_link0"/>
+      <parent link="wx200/base_link"/>
       <child link="camera_link"/>
   </joint>

File: intrarobots_ws/src/master/extrernal_urdfs/camera_depth.xacro (robot description, xacro)
@@ -4,8 +4,8 @@
       <axis xyz="0 1 0" />
       <!-- <origin rpy="0 ${pi/2} 0" xyz="0 0.54 0.8" /> -->
-      <origin rpy="${pi} ${3*pi/4} 0" xyz="0.4 0.3 0.35" />
+      <origin rpy="0 ${pi/4} 0" xyz="0 0 0.6" />
       <!--parent link fixed-->
-      <!-- <parent link="$(arg robot_name)/base_link"/> -->
-      <parent link="$(arg base_link_frame)"/>
+      <parent link="wx200/base_link"/>
+      <!-- <parent link="$(arg base_link_frame)"/> -->
       <child link="camera_link"/>
   </joint>
