Commit message: 1212

File: intrarobots_ws/src/master/extrernal_urdfs/camera_depth.xacro (robot description, xacro)
@@ -21,5 +21,5 @@
       <origin xyz="0 0 0" rpy="0 0 0"/>
       <geometry>
-        <box size="0.01 0.01 0.01"/>
+        <box size="0.01 0.03 0.03"/>
       </geometry>
     </collision>
